File: PCB/STM32 Led Controller.kicad_sch (KiCad schematic)
At the start: 66 parts, among them J1 EXT_PWR_CONN, J2 SWD_CONN, J3 12401610E4-2A, J4 WS2815, J5 RB1-125BAG1A, J6 Conn_02x04_Top_Bottom, SW1 FSM4JH, U1 Mini360, U2 NCV1117ST33T3G, U3 STM32G0B0RETx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

Commit message: minor tweaks, added logo, adjusted silkscreen
Parts:
- D1, D2: footprint Diode_SMD:D_SMB-SMC_Universal_Handsoldering -> Diode_SMD:D_SMA-SMB_Universal_Handsoldering
- R3, R4: value 100K -> 220
Connections:
- net +3V3: no longer R3.1
- net GND: now also D3.1 (K), U6.23 (RSVD)
- net TEST_LED: now also R3.1; no longer D3.1 (K)
- no-connect marks 61 -> 60
Other:
- moved on the sheet: D3, D4, R3, R4

Commit message: tweaked PCB, updated firmware
Parts:
- R3, R4: value 220 -> 330
Connections:
- net +3V3: now also R3.1
- net GND: no longer D3.1 (K), U6.23 (RSVD)
- net TEST_LED: now also D3.1 (K); no longer R3.1
- no-connect marks 60 -> 61
Other:
- moved on the sheet: D3, D4, J2, R3, R4
